File: PPG/PPG.sch (KiCad schematic (older format))
At the start: 53 parts

Commit message: Circuit Done
Parts:
- C1, C2, C4, C6, C7, C8: renamed from C?; footprint (none) -> Capacitor_SMD:C_0402_1005Metric
- C16, C17, C21, C24, C25, C26, C28, C29, C3, C30, C33, C34, C5: renamed from C?; footprint Capacitors_SMD:C_0402 -> Capacitor_SMD:C_0402_1005Metric
- C18: renamed from C?; footprint Capacitors_SMD:C_0402 -> Capacitor_SMD:C_0603_1608Metric
- C22, C23: renamed from C?; footprint Capacitors_SMD:C_0603 -> Capacitor_SMD:C_0603_1608Metric
- D1, D2, D3: renamed from D?; footprint (none) -> LED_SMD:LED_0603_1608Metric
- D4: renamed from D?; footprint LEDs:LED_0603 -> LED_SMD:LED_0603_1608Metric
- F1: renamed from F?; footprint (none) -> Capacitor_SMD:R_0402
- L1, L2, L4: renamed from L?; footprint (none) -> Inductor_SMD:L_0603_1608Metric
- L3, L5, L6: renamed from L?; footprint (none) -> Inductor_SMD:L_0402_1005Metric
- P1, P2, P3: renamed from J?; footprint (none) -> Connector_PinHeader_2.54mm:PinHeader_1x02_P2.54mm_Vertical
- R1, R2, R3: renamed from R?; footprint (none) -> Resistor_SMD:R_0402_1005Metric
- R10, R5, R7, R9: renamed from R?; footprint Resistors_SMD:R_0402 -> Resistor_SMD:R_0402_1005Metric
- U1: renamed from U?; footprint BGA8N40P2X4_87X156X50 -> Package_BGA:Texas_DSBGA-8_0.9x1.9mm_Layout2x4_P0.5mm
- U2: renamed from U?; footprint (none) -> Package_BGA:Texas_DSBGA-8_0.9x1.9mm_Layout2x4_P0.5mm
- U3: renamed from U?; footprint (none) -> Package_DFN_QFN:UQFN-48-1EP_6x6mm_Pitch0.4mm
- U6: renamed from U?; footprint (none) -> Package_DFN_QFN:DFN-8-1EP_2x3mm_P0.5mm_EP0.61x2.2mm
- gave numbers to parts that had none: 6
Connections:
- net DGND is gone; now on net GND: C1.2, C16.2, C17.2, C18.1, C2.2, C21.1, C22.2, C23.2, C24.1, C25.1, C26.2, C27.2, C28.2, C29.2, C3.2, C33.1, C34.2, C4.1, C5.2, C6.1, C7.1, C8.1, F1.1 (GND), F1.3 (GND), IC1.12 (GND), IC1.4 (PGND), L5.2, R10.2, R7.1, R9.2, U1.B2 (GND), U2.B2 (GND), U3.31 (VSS), U3.45 (VSS), U3.49 (THERMAL), U6.6 (Vss), U6.9 (EP_THRM), X1.2, X1.4
- net VccSwitch is gone; now on net LOAD_IN: C18.2, D4.1 (K), Q1.3 (S)
- net 1.8V: now also D1.2 (A)
- net 3.3V: no longer D1.2 (A)
- net MAX_INT(N): now also U3.22 (P0.19)
